File: CycleSync/Audio_ADC.kicad_sch (KiCad schematic)
At the start: 0 parts

Commit message: finished Phase 1.4
Parts:
- added C18, C20: 4u7, symbol Device:C
- added C19, C21: 0u01, symbol Device:C
- added C25, C27, C31, C34: 10u, symbol Device:C
- added C26, C28, C32, C33: 0u1, symbol Device:C
- added C30: 1u, symbol Device:C
- added D4, D5: D_TVS, symbol Device:D_TVS
- added R14, R17: 60k4, symbol Device:R
- added R15, R18: 20k, symbol Device:R
- added R16, R19: 100R, symbol Device:R
- added R20, R21: 0R, symbol Device:R
- added U3: PCM1862DBT, Package_SO:TSSOP-30_4.4x7.8mm_P0.5mm, symbol Audio:PCM1862DBT
Connections:
- net I2C_SCL: now also U3.24 (MC/SCL)
- net I2C_SDA: now also U3.23 (MOSI/SDA)
- new net: C19.2, R16.1, U3.3 (VINL1/VIN1P)
- new net: C18.2, R16.2
- new net: C18.1, R14.2, R15.2
- new net: C20.1, R17.2, R18.2
- new net: C20.2, R19.2
- new net: C33.2, C34.2, U3.11 (LDO)
- new net: R21.1, U3.25 (MS/AD)
- new net: R20.1, U3.26 (MD0)
- new net: C21.2, R19.1, U3.4 (VINR1/VIN2P)
- new net: C30.2, U3.6 (VREF)
- new net: D5.2 (A2), R17.1
- new net: D4.2 (A2), R14.1
- new net +3.3V: C25.2, C26.2, C27.2, C28.2, U3.13 (DVDD), U3.14 (IOVDD)
- new net +3V3: C31.2, C32.2, U3.8 (AVDD)
- new net GND: C19.1, C21.1, C25.1, C26.1, C27.1, C28.1, C30.1, C31.1, C32.1, C33.1, C34.1, D4.1 (A1), D5.1 (A1), R15.1, R18.1, R20.2, R21.2, U3.12 (DGND), U3.7 (AGND)
- no-connect marks 0 -> 5

Commit message: s
Parts:
- removed C19, C21: 0u01, symbol Device:C
- removed C20: 4u7, symbol Device:C
- removed C25, C27, C31, C34: 10u, symbol Device:C
- removed C28, C33: 0u1, symbol Device:C
- removed C30: 1u, symbol Device:C
- removed D5: D_TVS, symbol Device:D_TVS
- removed R16, R19: 100R, symbol Device:R
- removed R17: 60k4, symbol Device:R
- removed R18: 20k, symbol Device:R
- removed R20, R21: 0R, symbol Device:R
- added C40, C42: 220p, Capacitor_SMD:C_0603_1608Metric, symbol Device:C
- added C41: 10u, Capacitor_SMD:C_0603_1608Metric, symbol Device:C
- added C44, C46, C49: 10u, symbol Device:C
- added C45: 0u1, symbol Device:C
- added C47: 1u, symbol Device:C
- added D8: PESD24VL1BA, Diode_SMD:D_SOD-323, symbol Device:D_TVS
- added R27, R30: 47R, symbol Device:R
- added R28: 60k4, symbol Device:R
- added R29: 19k6, symbol Device:R
- C39: renamed from C18; value 4u7 -> 10u; footprint (none) -> Capacitor_SMD:C_0603_1608Metric; Variant (none) -> LINE_IN_OPTION
- C43: renamed from C32; Variant (none) -> LINE_IN_OPTION
- C48: renamed from C26; Variant (none) -> LINE_IN_OPTION
- D4: value D_TVS -> PESD24VL1BA; footprint (none) -> Diode_SMD:D_SOD-323; Variant (none) -> LINE_IN_OPTION
- R25: renamed from R14; Variant (none) -> LINE_IN_OPTION
- R26: renamed from R15; value 20k -> 19k6; Variant (none) -> LINE_IN_OPTION
- U3: Variant (none) -> LINE_IN_OPTION
Connections:
- net GND: now also U3.25 (MS/AD), U3.26 (MD0), C40.1, C42.1, C44.1, C45.1, C46.1, C47.1, C49.1, D8.1 (A1), R29.1
- net I2S_BCK: now also U3.17 (BCK)
- net I2S_DIN: now also U3.18 (DOUT)
- net I2S_LRCK: now also U3.16 (LRCK)
- net ADC_IN_L: now reaches U3.3 (VINL1/VIN1P)
- net ADC_IN_L: now also C40.2, R27.2
- net LINE_L_AC: now reaches C39.2
- net LINE_L_AC: now also R27.1
- net LINE_L_ATTEN: now reaches C39.1, R25.2, R26.2
- net at U3.11 (LDO): now also C45.2, C46.2
- net ADC_IN_R: now reaches U3.4 (VINR1/VIN2P)
- net ADC_IN_R: now also C42.2, R30.2
- net at U3.6 (VREF): now also C47.2
- net LINE_IN_L: now reaches D4.2 (A2), R25.1
- net +3.3V renamed +3V3_DIG
- net +3V3_DIG: now also C49.2
- net +3V3 renamed +3V3_AUDIO
- net +3V3_AUDIO: now also C44.2
- new net LINE_IN_R: D8.2 (A2), R28.1
- new net LINE_R_AC: C41.2, R30.1
- new net LINE_R_ATTEN: C41.1, R28.2, R29.2
- no-connect marks 5 -> 14
Other:
- note added: "ADC CONFIGURATION MD0 = LOW: I²C CONTROL MODE MS/AD = LOW: 7-BIT I²C ADDRESS 0x4A I²C1 PULL-UP PAIR IS SELECTED BY THE PD VARIANT; SEE MCU AND USB_PD SHEETS. I²S SLAVE; BCK PLL MODE IS USED WHEN SCKI IS ABSENT. TARGET AUDIO FORMAT: 48 kHz / 24-BIT."
- note added: "ANALOG SUPPLY DECOUPLING"
- note added: "CONTROL MODE & I²C ADDRESS STRAPS"
- note added: "DIGITAL SUPPLY DECOUPLING"
- note added: "I²S OUTPUT & I²C CONTROL"
- note added: "OPTIONAL LINE-IN / ADC ASSEMBLY — DNP AS COMPLETE GROUP"
- note added: "OPTIONAL LINE-IN / ADC POPULATION GROUP LINE-IN BUILD: POPULATE U3, R25-R30, C39-C49, D4, D8, PLUS J5 AND D5 ON DAUGHTER_IO. PLAYBACK-ONLY BUILD: DNP ALL COMPONENTS LISTED ABOVE. VARIANT FIELD = LINE_IN_OPTION I2C PULL-UP SELECTION IS CONTROLLED SEPARATELY BY THE PD / NO-PD OPTION."
- note added: "PCM1862 STEREO AUDIO ADC"
- note added: "STEREO LINE-IN PROTECTION, ATTENUATION & AC COUPLING"
- note added: "internal LDO output in 3.3-V mode; symbol pin is dual-purpose."
- title: (none) -> PCM1862 STEREO AUDIO ADC & OPTIONAL LINE INPUT
- moved on the sheet: C39, C43, C48, D4, R25, R26, U3

Commit message: verified schematic wirings
Parts:
- C48: renamed from C40; value 220p -> 1n5
- C50: renamed from C42; value 220p -> 1n5
- R27: renamed from R25; value 60k4 -> 1k30
- R28: renamed from R26; value 19k6 -> 1k58
- R29: renamed from R27; value 47R -> 100R
- R30: renamed from R28; value 60k4 -> 1k30
- R31: renamed from R29; value 19k6 -> 1k58
- R32: renamed from R30; value 47R -> 100R
- renumbered C43 to C40, C44 to C41, C45 to C42, C46 to C43, C47 to C44, C48 to C45, C49 to C46, C39 to C47, C41 to C49, D8 to D5, U3 to U6
Other:
- note added: "LINE-IN FRONT END - EACH CHANNEL DAUGHTER R56/R57 = 10 kΩ MAIN R27/R30 = 1.30 kΩ SERIES R28/R31 = 1.58 kΩ SHUNT R29/R32 = 100 Ω ADC SERIES C47/C49 = 10 µF; C48/C50 = 1.5 nF ASSUMING 100 Ω SOURCE AND 20 kΩ ADC INPUT: GAIN ≈ -18.9 dB AT 1 kHz. +26 dBu INPUT → ≈ 1.75 Vrms AT ADC. WORST CASE ≈ 2.05 Vrms < 2.1 Vrms FULL SCALE."
- note added: "OPTIONAL LINE-IN / ADC POPULATION GROUP LINE-IN BUILD: POPULATE U6, R27-R32, C40-C50, D4 AND D5; PLUS J5, D11, R56 AND R57 ON DAUGHTER_IO. PLAYBACK-ONLY BUILD: DNP ALL COMPONENTS LISTED ABOVE. VARIANT FIELD = LINE_IN_OPTION. I²C PULL-UP SELECTION IS CONTROLLED BY THE PD / NO-PD VARIANT."
- note removed: "OPTIONAL LINE-IN / ADC POPULATION GROUP LINE-IN BUILD: POPULATE U3, R25-R30, C39-C49, D4, D8, PLUS J5 AND D5 ON DAUGHTER_IO. PLAYBACK-ONLY BUILD: DNP ALL COMPONENTS LISTED ABOVE. VARIANT FIELD = LINE_IN_OPTION I2C PULL-UP SELECTION IS CONTROLLED SEPARATELY BY THE PD / NO-PD OPTION."
Changed lines of the file:
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@@
 	)
 	(rectangle
-		(start 20.32 134.62)
-		(end 77.47 156.21)
+		(start 207.518 118.11)
+		(end 263.398 143.51)
+		(stroke
+			(width 0)
+			(type default)
+		)
+		(fill
+			(type none)
+		)
+	)
+	(rectangle
+		(start 19.558 137.668)
+		(end 76.708 159.258)
 		(stroke
 			(width 0)
@@
 	(text "ADC CONFIGURATION\n\nMD0 = LOW: I²C CONTROL MODE\nMS/AD = LOW: 7-BIT I²C ADDRESS 0x4A\n\nI²C1 PULL-UP PAIR IS SELECTED BY THE PD VARIANT;\nSEE MCU AND USB_PD SHEETS.\n\nI²S SLAVE; BCK PLL MODE IS USED WHEN SCKI IS ABSENT.\nTARGET AUDIO FORMAT: 48 kHz / 24-BIT."
 		(exclude_from_sim no)
-		(at 49.022 145.542 0)
+		(at 48.26 148.59 0)
 		(effects
 			(font
@@
 		)
 	)
-	(text "OPTIONAL LINE-IN / ADC POPULATION GROUP\n\nLINE-IN BUILD:\nPOPULATE U3, R25-R30, C39-C49,\nD4, D8, PLUS J5 AND D5 ON DAUGHTER_IO.\n\nPLAYBACK-ONLY BUILD:\nDNP ALL COMPONENTS LISTED ABOVE.\n\nVARIANT FIELD = LINE_IN_OPTION\nI2C PULL-UP SELECTION IS CONTROLLED SEPARATELY\nBY THE PD / NO-PD OPTION."
+	(text "OPTIONAL LINE-IN / ADC POPULATION GROUP\n\nLINE-IN BUILD:\nPOPULATE U6, R27-R32, C40-C50, D4 AND D5;\nPLUS J5, D11, R56 AND R57 ON DAUGHTER_IO.\n\nPLAYBACK-ONLY BUILD:\nDNP ALL COMPONENTS LISTED ABOVE.\n\nVARIANT FIELD = LINE_IN_OPTION.\nI²C PULL-UP SELECTION IS CONTROLLED BY\nTHE PD / NO-PD VARIANT."
 		(exclude_from_sim no)
 		(at 54.102 35.814 0)
@@
 		)
 	)
+	(text "LINE-IN FRONT END - EACH CHANNEL\n\nDAUGHTER R56/R57 = 10 kΩ\nMAIN R27/R30 = 1.30 kΩ SERIES\nR28/R31 = 1.58 kΩ SHUNT\nR29/R32 = 100 Ω ADC SERIES\nC47/C49 = 10 µF; C48/C50 = 1.5 nF\n\nASSUMING 100 Ω SOURCE AND 20 kΩ ADC INPUT:\nGAIN ≈ -18.9 dB AT 1 kHz.\n+26 dBu INPUT → ≈ 1.75 Vrms AT ADC.\nWORST CASE ≈ 2.05 Vrms < 2.1 Vrms FULL SCALE."
+		(exclude_from_sim no)
+		(at 236.22 130.81 0)
+		(effects
+			(font
+				(size 1.27 1.27)
+			)
+		)
+	)
 	(text "PCM1862 STEREO AUDIO ADC"
 		(exclude_from_sim no)
-		(at 149.098 134.874 0)
+		(at 147.32 132.588 0)
 		(effects
 			(font
@@
 		(dnp no)
 		(fields_autoplaced yes)
-		(property "Reference" "C48"
+		(property "Reference" "C45"
 			(at 212.09 45.7199 0)
 			(show_name no)
@@
 			(project "CycleSync"
 				(path "/3f2cc6af-e67b-48ad-b391-ff7619611bd8/f6d46258-8d13-4c87-b95e-4a5b8c76ac66"
-					(reference "C48")
+					(reference "C45")
 					(unit 1)
 				)
@@
 		(dnp no)
 		(fields_autoplaced yes)
-		(property "Reference" "C39"
+		(property "Reference" "C47"
 			(at 99.06 76.2 90)
 			(show_name no)
@@
 			(project "CycleSync"
 				(path "/3f2cc6af-e67b-48ad-b391-ff7619611bd8/f6d46258-8d13-4c87-b95e-4a5b8c76ac66"
-					(reference "C39")
+					(reference "C47")
 					(unit 1)
 				)
@@
 		(dnp no)
 		(fields_autoplaced yes)
-		(property "Reference" "R28"
+		(property "Reference" "R30"
 			(at 74.93 101.6 90)
 			(show_name no)
@@
 			)
 		)
-		(property "Value" "60k4"
+		(property "Value" "1k30"
 			(at 74.93 104.14 90)
 			(show_name no)
@@
 			(project "CycleSync"
 				(path "/3f2cc6af-e67b-48ad-b391-ff7619611bd8/f6d46258-8d13-4c87-b95e-4a5b8c76ac66"
-					(reference "R28")
+					(reference "R30")
 					(unit 1)
 				)
@@
 		(dnp no)
 		(fields_autoplaced yes)
-		(property "Reference" "C43"
+		(property "Reference" "C40"
 			(at 134.62 45.7199 0)
 			(show_name no)
@@
 			(project "CycleSync"
 				(path "/3f2cc6af-e67b-48ad-b391-ff7619611bd8/f6d46258-8d13-4c87-b95e-4a5b8c76ac66"
-					(reference "C43")
+					(reference "C40")
 					(unit 1)
 				)
@@
 		(dnp no)
 		(fields_autoplaced yes)
-		(property "Reference" "R29"
+		(property "Reference" "R31"
 			(at 83.82 111.7599 0)
 			(show_name no)
@@
 			)
 		)
-		(property "Value" "19k6"
+		(property "Value" "1k58"
 			(at 83.82 114.2999 0)
 			(show_name no)
@@
 			(project "CycleSync"
 				(path "/3f2cc6af-e67b-48ad-b391-ff7619611bd8/f6d46258-8d13-4c87-b95e-4a5b8c76ac66"
-					(reference "R29")
+					(reference "R31")
 					(unit 1)
 				)
@@
 		(dnp no)
 		(fields_autoplaced yes)
-		(property "Reference" "R27"
+		(property "Reference" "R29"
 			(at 120.65 77.47 90)
 			(show_name no)
@@
 			)
 		)
-		(property "Value" "47R"
+		(property "Value" "100R"
 			(at 120.65 80.01 90)
 			(show_name no)
@@
 			(project "CycleSync"
 				(path "/3f2cc6af-e67b-48ad-b391-ff7619611bd8/f6d46258-8d13-4c87-b95e-4a5b8c76ac66"
-					(reference "R27")
+					(reference "R29")
 					(unit 1)
 				)
@@
 		(dnp no)
 		(fields_autoplaced yes)
-		(property "Reference" "D8"
+		(property "Reference" "D5"
 			(at 64.77 113.0299 90)
 			(show_name no)
@@
 			(project "CycleSync"
 				(path "/3f2cc6af-e67b-48ad-b391-ff7619611bd8/f6d46258-8d13-4c87-b95e-4a5b8c76ac66"
-					(reference "D8")
+					(reference "D5")
 					(unit 1)
 				)
@@
 		(dnp no)
 		(fields_autoplaced yes)
-		(property "Reference" "C46"
+		(property "Reference" "C43"
 			(at 193.04 55.8799 0)
 			(show_name no)
@@
 			(project "CycleSync"
 				(path "/3f2cc6af-e67b-48ad-b391-ff7619611bd8/f6d46258-8d13-4c87-b95e-4a5b8c76ac66"
-					(reference "C46")
+					(reference "C43")
 					(unit 1)
 				)
@@
 		(in_pos_files yes)
 		(dnp no)
-		(property "Reference" "U3"
-			(at 172.3233 133.35 0)
+		(property "Reference" "U6"
+			(at 176.784 73.406 0)
 			(show_name no)
 			(do_not_autoplace no)
@@
 		)
 		(property "Value" "PCM1862DBT"
-			(at 172.3233 135.89 0)
+			(at 172.212 132.588 0)
 			(show_name no)
 			(do_not_autoplace no)
@@
 			(project "CycleSync"
 				(path "/3f2cc6af-e67b-48ad-b391-ff7619611bd8/f6d46258-8d13-4c87-b95e-4a5b8c76ac66"
-					(reference "U3")
+					(reference "U6")
 					(unit 1)
 				)
@@
 		(dnp no)
 		(fields_autoplaced yes)
-		(property "Reference" "C47"
+		(property "Reference" "C44"
 			(at 209.55 66.0399 0)
 			(show_name no)
@@
 			(project "CycleSync"
 				(path "/3f2cc6af-e67b-48ad-b391-ff7619611bd8/f6d46258-8d13-4c87-b95e-4a5b8c76ac66"
-					(reference "C47")
+					(reference "C44")
 					(unit 1)
 				)
@@
 		(dnp no)
 		(fields_autoplaced yes)
-		(property "Reference" "C42"
+		(property "Reference" "C50"
 			(at 135.89 114.2999 0)
 			(show_name no)
@@
 			)
 		)
-		(property "Value" "220p"
+		(property "Value" "1n5"
 			(at 135.89 116.8399 0)
 			(show_name no)
@@
 			(project "CycleSync"
 				(path "/3f2cc6af-e67b-48ad-b391-ff7619611bd8/f6d46258-8d13-4c87-b95e-4a5b8c76ac66"
-					(reference "C42")
+					(reference "C50")
 					(unit 1)
 				)
@@
 		(dnp no)
 		(fields_autoplaced yes)
-		(property "Reference" "C44"
+		(property "Reference" "C41"
 			(at 147.32 45.7199 0)
 			(show_name no)
@@
 			(project "CycleSync"
 				(path "/3f2cc6af-e67b-48ad-b391-ff7619611bd8/f6d46258-8d13-4c87-b95e-4a5b8c76ac66"
-					(reference "C44")
+					(reference "C41")
 					(unit 1)
 				)
@@
 		(dnp no)
 		(fields_autoplaced yes)
-		(property "Reference" "C41"
+		(property "Reference" "C49"
 			(at 101.6 100.33 90)
 			(show_name no)
@@
 			(project "CycleSync"
 				(path "/3f2cc6af-e67b-48ad-b391-ff7619611bd8/f6d46258-8d13-4c87-b95e-4a5b8c76ac66"
-					(reference "C41")
+					(reference "C49")
 					(unit 1)
 				)
@@
 		(dnp no)
 		(fields_autoplaced yes)
-		(property "Reference" "R26"
+		(property "Reference" "R28"
 			(at 83.82 87.6299 0)
 			(show_name no)
@@
 			)
 		)
-		(property "Value" "19k6"
+		(property "Value" "1k58"
 			(at 83.82 90.1699 0)
 			(show_name no)
@@
 			(project "CycleSync"
 				(path "/3f2cc6af-e67b-48ad-b391-ff7619611bd8/f6d46258-8d13-4c87-b95e-4a5b8c76ac66"
-					(reference "R26")
+					(reference "R28")
 					(unit 1)
 				)
@@
 		(dnp no)
 		(fields_autoplaced yes)
-		(property "Reference" "R25"
+		(property "Reference" "R27"
 			(at 74.93 77.47 90)
 			(show_name no)
@@
 			)
 		)
-		(property "Value" "60k4"
+		(property "Value" "1k30"
 			(at 74.93 80.01 90)
 			(show_name no)
@@
 			(project "CycleSync"
 				(path "/3f2cc6af-e67b-48ad-b391-ff7619611bd8/f6d46258-8d13-4c87-b95e-4a5b8c76ac66"
-					(reference "R25")
+					(reference "R27")
 					(unit 1)
 				)
@@
 		(dnp no)
 		(fields_autoplaced yes)
-		(property "Reference" "R30"
+		(property "Reference" "R32"
 			(at 121.92 101.6 90)
 			(show_name no)
@@
 			)
 		)
-		(property "Value" "47R"
+		(property "Value" "100R"
 			(at 121.92 104.14 90)
 			(show_name no)
@@
 			(project "CycleSync"
 				(path "/3f2cc6af-e67b-48ad-b391-ff7619611bd8/f6d46258-8d13-4c87-b95e-4a5b8c76ac66"
-					(reference "R30")
+					(reference "R32")
 					(unit 1)
 				)
@@
 		(dnp no)
 		(fields_autoplaced yes)
-		(property "Reference" "C40"
+		(property "Reference" "C48"
 			(at 135.89 88.8999 0)
 			(show_name no)
@@
 			)
 		)
-		(property "Value" "220p"
+		(property "Value" "1n5"
 			(at 135.89 91.4399 0)
 			(show_name no)
@@
 			(project "CycleSync"
 				(path "/3f2cc6af-e67b-48ad-b391-ff7619611bd8/f6d46258-8d13-4c87-b95e-4a5b8c76ac66"
-					(reference "C40")
+					(reference "C48")
 					(unit 1)
 				)
@@
 		(dnp no)
 		(fields_autoplaced yes)
-		(property "Reference" "C49"
+		(property "Reference" "C46"
 			(at 223.52 45.7199 0)
 			(show_name no)
@@
 			(project "CycleSync"
 				(path "/3f2cc6af-e67b-48ad-b391-ff7619611bd8/f6d46258-8d13-4c87-b95e-4a5b8c76ac66"
-					(reference "C49")
+					(reference "C46")
 					(unit 1)
 				)
@@
 		(dnp no)
 		(fields_autoplaced yes)
-		(property "Reference" "C45"
+		(property "Reference" "C42"
 			(at 182.88 55.8799 0)
 			(show_name no)
@@
 			(project "CycleSync"
 				(path "/3f2cc6af-e67b-48ad-b391-ff7619611bd8/f6d46258-8d13-4c87-b95e-4a5b8c76ac66"
-					(reference "C45")
+					(reference "C42")
 					(unit 1)
 				)

Commit message: added some new testpoints for I2C
Parts:
- added TP14: I2S_DIN, TestPoint:TestPoint_Pad_D1.5mm, symbol Connector:TestPoint
- C40, C42, C45: footprint (none) -> Capacitor_SMD:C_0402_1005Metric
- C41, C43, C46: footprint (none) -> Capacitor_SMD:C_0805_2012Metric
- C44: footprint (none) -> Capacitor_SMD:C_0603_1608Metric
- C47, C49: footprint Capacitor_SMD:C_0603_1608Metric -> Capacitor_SMD:C_0805_2012Metric
- R27, R28, R29, R30, R31, R32: footprint (none) -> Resistor_SMD:R_0603_1608Metric
Connections:
- net I2S_DIN: now also TP14.1
Changed lines of the file:
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@@
 	(text "I²S OUTPUT & I²C CONTROL"
 		(exclude_from_sim no)
-		(at 218.948 89.662 0)
+		(at 270.002 97.79 0)
 		(effects
 			(font
@@
 		(color 0 0 0 0)
 	)
+	(junction
+		(at 214.63 92.71)
+		(diameter 0)
+		(color 0 0 0 0)
+	)
 	(no_connect
 		(at 152.4 113.03)
@@
 	(wire
 		(pts
+			(xy 214.63 92.71) (xy 226.06 92.71)
+		)
+		(stroke
+			(width 0)
+			(type default)
+		)
+	)
+	(wire
+		(pts
 			(xy 167.64 69.85) (xy 165.1 69.85)
 		)
@@
 	(wire
 		(pts
-			(xy 182.88 92.71) (xy 190.5 92.71)
+			(xy 182.88 92.71) (xy 214.63 92.71)
 		)
 		(stroke
@@
 	(hierarchical_label "I2S_DIN"
 		(shape output)
-		(at 190.5 92.71 0)
+		(at 226.06 92.71 0)
 		(effects
 			(font
@@
 			)
 		)
-		(property "Footprint" ""
+		(property "Footprint" "Capacitor_SMD:C_0402_1005Metric"
 			(at 207.3148 43.18 0)
 			(hide yes)
@@
 			)
 		)
-		(property "Footprint" "Capacitor_SMD:C_0603_1608Metric"
+		(property "Footprint" "Capacitor_SMD:C_0805_2012Metric"
 			(at 102.87 82.8548 0)
 			(hide yes)
@@
 	)
 	(symbol
+		(lib_id "Connector:TestPoint")
+		(at 214.63 92.71 0)
+		(unit 1)
+		(body_style 1)
+		(exclude_from_sim no)
+		(in_bom yes)
+		(on_board yes)
+		(in_pos_files yes)
+		(dnp no)
+		(fields_autoplaced yes)
+		(property "Reference" "TP14"
+			(at 217.17 88.1379 0)
+			(show_name no)
+			(do_not_autoplace no)
+			(effects
+				(font
+					(size 1.27 1.27)
+				)
+				(justify left)
+			)
+		)
+		(property "Value" "I2S_DIN"
+			(at 217.17 90.6779 0)
+			(show_name no)
+			(do_not_autoplace no)
+			(effects
+				(font
+					(size 1.27 1.27)
+				)
+				(justify left)
+			)
+		)
+		(property "Footprint" "TestPoint:TestPoint_Pad_D1.5mm"
+			(at 219.71 92.71 0)
+			(hide yes)
+			(show_name no)
+			(do_not_autoplace no)
+			(effects
+				(font
+					(size 1.27 1.27)
+				)
+			)
+		)
+		(property "Datasheet" ""
+			(at 219.71 92.71 0)
+			(hide yes)
+			(show_name no)
+			(do_not_autoplace no)
+			(effects
+				(font
+					(size 1.27 1.27)
+				)
+			)
+		)
+		(property "Description" "test point"
+			(at 214.63 92.71 0)
+			(hide yes)
+			(show_name no)
+			(do_not_autoplace no)
+			(effects
+				(font
+					(size 1.27 1.27)
+				)
+			)
+		)
+		(pin "1"
+		)
+		(instances
+			(project "CycleSync"
+				(path "/3f2cc6af-e67b-48ad-b391-ff7619611bd8/f6d46258-8d13-4c87-b95e-4a5b8c76ac66"
+					(reference "TP14")
+					(unit 1)
+				)
+			)
+		)
+	)
+	(symbol
 		(lib_id "Device:R")
 		(at 74.93 107.95 90)
@@
 			)
 		)
-		(property "Footprint" ""
+		(property "Footprint" "Resistor_SMD:R_0603_1608Metric"
 			(at 74.93 109.728 90)
 			(hide yes)
@@
 			)
 		)
-		(property "Footprint" ""
+		(property "Footprint" "Capacitor_SMD:C_0402_1005Metric"
 			(at 129.8448 43.18 0)
 			(hide yes)
@@
 			)
 		)
-		(property "Footprint" ""
+		(property "Footprint" "Resistor_SMD:R_0603_1608Metric"
 			(at 83.058 113.03 90)
 			(hide yes)
@@
 			)
 		)
-		(property "Footprint" ""
+		(property "Footprint" "Resistor_SMD:R_0603_1608Metric"
 			(at 120.65 85.598 90)
 			(hide yes)
@@
 			)
 		)
-		(property "Footprint" ""
+		(property "Footprint" "Capacitor_SMD:C_0805_2012Metric"
 			(at 188.2648 53.34 0)
 			(hide yes)
@@
 			)
 		)
-		(property "Footprint" ""
+		(property "Footprint" "Capacitor_SMD:C_0603_1608Metric"
 			(at 204.7748 63.5 0)
 			(hide yes)
@@
 			)
 		)
-		(property "Footprint" ""
+		(property "Footprint" "Capacitor_SMD:C_0805_2012Metric"
 			(at 142.5448 43.18 0)
 			(hide yes)
@@
 			)
 		)
-		(property "Footprint" "Capacitor_SMD:C_0603_1608Metric"
+		(property "Footprint" "Capacitor_SMD:C_0805_2012Metric"
 			(at 105.41 106.9848 0)
 			(hide yes)
@@
 			)
 		)
-		(property "Footprint" ""
+		(property "Footprint" "Resistor_SMD:R_0603_1608Metric"
 			(at 83.058 88.9 90)
 			(hide yes)
@@
 			)
 		)
-		(property "Footprint" ""
+		(property "Footprint" "Resistor_SMD:R_0603_1608Metric"
 			(at 74.93 85.598 90)
 			(hide yes)
@@
 			)
 		)
-		(property "Footprint" ""
+		(property "Footprint" "Resistor_SMD:R_0603_1608Metric"
 			(at 121.92 109.728 90)
 			(hide yes)
@@
 			)
 		)
-		(property "Footprint" ""
+		(property "Footprint" "Capacitor_SMD:C_0805_2012Metric"
 			(at 218.7448 43.18 0)
 			(hide yes)
@@
 			)
 		)
-		(property "Footprint" ""
+		(property "Footprint" "Capacitor_SMD:C_0402_1005Metric"
 			(at 178.1048 53.34 0)
 			(hide yes)
