File: CycleSync/Audio_DAC.kicad_sch (KiCad schematic)
At the start: 0 parts

Commit message: finished Phase 1.4
Parts:
- added C29, C35, C38, C41: 0u1, symbol Device:C
- added C36, C37, C39, C40: 10u, symbol Device:C
- added C42: 2u2, symbol Device:C
- added C43, C44: 2n2, symbol Device:C
- added C45, C46: 1u, symbol Device:C
- added R22, R23, R24, R25: 0R, symbol Device:R
- added R26, R27: 470R, symbol Device:R
- added U4: PCM5102A, Package_SO:TSSOP-20_4.4x6.5mm_P0.65mm, symbol Audio:PCM5102A
Connections:
- net I2S_BCK: now also U4.13 (BCK)
- net I2S_DOUT: now also U4.14 (DIN)
- net I2S_LRCK: now also U4.15 (LRCK)
- new net: C43.1, C46.1, R26.2
- new net: R24.2, U4.11 (FLT)
- new net: C29.1, C37.1, C38.1, C39.1
- new net: R27.1, U4.6 (OUTL)
- new net: C44.1, C45.1, R27.2
- new net: C41.2, U4.18 (LDOO)
- new net: R22.2, U4.12 (SCK)
- new net: C40.2, U4.5 (VNEG)
- new net: R23.2, U4.16 (FMT)
- new net: R26.1, U4.7 (OUTR)
- new net: C42.1, U4.2 (CAPP)
- new net: C42.2, U4.4 (CAPM)
- new net: R25.2, U4.10 (DEMP)
- new net +3.3V: C29.2, C37.2, C38.2, C39.2, U4.1 (CPVDD), U4.20 (DVDD)
- new net +3V3: C35.2, C36.2
- new net AVDD: C35.1, C36.1, U4.17 (XSMT), U4.8 (AVDD)
- new net GND: C40.1, C41.1, C43.2, C44.2, R22.1, R23.1, R24.1, R25.1, U4.19 (DGND), U4.3 (CPGND), U4.9 (AGND)
- new net LINE_OUT_L: C45.2
- new net LINE_OUT_R: C46.2

Commit message: s
Parts:
- removed C35, C38: 0u1, symbol Device:C
- removed C36, C39: 10u, symbol Device:C
- removed R22, R23, R24, R25: 0R, symbol Device:R
- added C27, C29, C34: 0u1, symbol Device:C
- added C28, C30: 10u, symbol Device:C
- added TP12, TP13, TP14: TestPoint, symbol Connector:TestPoint
- C32: renamed from C40; value 10u -> 2u2
- C33: renamed from C41; value 0u1 -> 10u
- C36: renamed from C45; value 1u -> 4u7
- C38: renamed from C46; value 1u -> 4u7
- renumbered C29 to C25, C37 to C26, C42 to C31, C44 to C35, C43 to C37, R27 to R23, R26 to R24
Connections:
- net AVDD is gone; now on net +3V3_AUDIO: U4.17 (XSMT), U4.8 (AVDD)
- net GND: now also C25.1, C26.1, C33.2, U4.10 (DEMP), U4.11 (FLT), U4.12 (SCK), U4.16 (FMT), C27.1, C28.1, C29.1, C30.1, C34.2; no longer C33.1
- net I2S_BCK: now also TP14.1
- net I2S_DOUT: now also TP13.1
- net I2S_LRCK: now also TP12.1
- net OUT_R_FILTERED: now reaches C37.1, C38.1, R24.2
- net OUT_L_RAW: now reaches R23.1, U4.6 (OUTL)
- net OUT_L_FILTERED: now reaches C35.1, C36.1, R23.2
- net LDO_OUT: now reaches U4.18 (LDOO)
- net LDO_OUT: now also C33.1, C34.1; no longer C33.2
- net VNEG: now reaches C32.2, U4.5 (VNEG)
- net OUT_R_RAW: now reaches R24.1, U4.7 (OUTR)
- net CP_FLY_P: now reaches C31.1, U4.2 (CAPP)
- net CP_FLY_M: now reaches C31.2, U4.4 (CAPM)
- net +3.3V renamed +3V3_AUDIO
- net +3V3_AUDIO: now also C27.2, C28.2; no longer U4.20 (DVDD)
- new net +3V3_DIG: C29.2, C30.2, U4.20 (DVDD)
Other:
- note added: "ANALOG & DIGITAL SUPPLY DECOUPLING"
- note added: "I²S INPUT — MCU MASTER / DAC SLAVE"
- note added: "STEREO OUTPUT FILTER & AC COUPLING"
- note added: "U4 HARDWARE CONFIGURATION SCK = LOW: 3-WIRE I²S; INTERNAL PLL USES BCK. FMT = LOW: I²S DATA FORMAT. FLT = LOW: NORMAL-LATENCY FILTER. DEMP = LOW: DE-EMPHASIS DISABLED. XSMT = HIGH: HARDWARE MUTE IS NOT MCU-CONTROLLED. NO EXTERNAL MCLK OR I²C CONTROL."
- title: (none) -> PCM5102A I²S DAC & STEREO LINE OUTPUT
- moved on the sheet: C25, C26, C31, C32, C33, C35, C36, C37, C38, R23, R24, U4

Commit message: verified schematic wirings
Parts:
- renumbered C25 to C26, C26 to C27, C27 to C28, C28 to C29, C29 to C30, C30 to C31, C31 to C32, C32 to C33, C33 to C34, C34 to C35, C35 to C36, C36 to C37, C37 to C38, C38 to C39, R24 to R25, R23 to R26, U4 to U5
Other:
- note added: "C37/C39: 4.7 µF NON-POLAR LINE-OUTPUT AC-COUPLING CAPACITORS."
Changed lines of the file:
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@@
 		)
 	)
+	(text "C37/C39: 4.7 µF NON-POLAR\nLINE-OUTPUT AC-COUPLING CAPACITORS."
+		(exclude_from_sim no)
+		(at 252.73 97.028 0)
+		(effects
+			(font
+				(size 1.27 1.27)
+			)
+		)
+	)
 	(text "I²S INPUT — MCU MASTER / DAC SLAVE"
 		(exclude_from_sim no)
@@
 		(dnp no)
 		(fields_autoplaced yes)
-		(property "Reference" "C37"
+		(property "Reference" "C38"
 			(at 204.47 114.2999 0)
 			(show_name no)
@@
 			(project "CycleSync"
 				(path "/3f2cc6af-e67b-48ad-b391-ff7619611bd8/b5b9e253-8b7f-4bb9-bef8-83286ffed738"
-					(reference "C37")
+					(reference "C38")
 					(unit 1)
 				)
@@
 		(dnp no)
 		(fields_autoplaced yes)
-		(property "Reference" "C26"
+		(property "Reference" "C27"
 			(at 95.25 74.9299 0)
 			(show_name no)
@@
 			(project "CycleSync"
 				(path "/3f2cc6af-e67b-48ad-b391-ff7619611bd8/b5b9e253-8b7f-4bb9-bef8-83286ffed738"
-					(reference "C26")
+					(reference "C27")
 					(unit 1)
 				)
@@
 		(dnp no)
 		(fields_autoplaced yes)
-		(property "Reference" "C29"
+		(property "Reference" "C30"
 			(at 143.51 71.1199 0)
 			(show_name no)
@@
 			(project "CycleSync"
 				(path "/3f2cc6af-e67b-48ad-b391-ff7619611bd8/b5b9e253-8b7f-4bb9-bef8-83286ffed738"
-					(reference "C29")
+					(reference "C30")
 					(unit 1)
 				)
@@
 		(dnp no)
 		(fields_autoplaced yes)
-		(property "Reference" "C38"
+		(property "Reference" "C39"
 			(at 215.9 101.6 90)
 			(show_name no)
@@
 			(project "CycleSync"
 				(path "/3f2cc6af-e67b-48ad-b391-ff7619611bd8/b5b9e253-8b7f-4bb9-bef8-83286ffed738"
-					(reference "C38")
+					(reference "C39")
 					(unit 1)
 				)
@@
 		(dnp no)
 		(fields_autoplaced yes)
-		(property "Reference" "C25"
+		(property "Reference" "C26"
 			(at 85.09 74.9299 0)
 			(show_name no)
@@
 			(project "CycleSync"
 				(path "/3f2cc6af-e67b-48ad-b391-ff7619611bd8/b5b9e253-8b7f-4bb9-bef8-83286ffed738"
-					(reference "C25")
+					(reference "C26")
 					(unit 1)
 				)
@@
 		(dnp no)
 		(fields_autoplaced yes)
-		(property "Reference" "R23"
+		(property "Reference" "R26"
 			(at 199.39 77.47 90)
 			(show_name no)
@@
 			(project "CycleSync"
 				(path "/3f2cc6af-e67b-48ad-b391-ff7619611bd8/b5b9e253-8b7f-4bb9-bef8-83286ffed738"
-					(reference "R23")
+					(reference "R26")
 					(unit 1)
 				)
@@
 		(in_pos_files yes)
 		(dnp no)
-		(property "Reference" "C33"
+		(property "Reference" "C34"
 			(at 166.37 123.698 0)
 			(show_name no)
@@
 			(project "CycleSync"
 				(path "/3f2cc6af-e67b-48ad-b391-ff7619611bd8/b5b9e253-8b7f-4bb9-bef8-83286ffed738"
-					(reference "C33")
+					(reference "C34")
 					(unit 1)
 				)
@@
 		(in_pos_files yes)
 		(dnp no)
-		(property "Reference" "C32"
+		(property "Reference" "C33"
 			(at 149.86 120.65 90)
 			(show_name no)
@@
 			(project "CycleSync"
 				(path "/3f2cc6af-e67b-48ad-b391-ff7619611bd8/b5b9e253-8b7f-4bb9-bef8-83286ffed738"
-					(reference "C32")
+					(reference "C33")
 					(unit 1)
 				)
@@
 		(dnp no)
 		(fields_autoplaced yes)
-		(property "Reference" "R24"
+		(property "Reference" "R25"
 			(at 181.61 102.87 90)
 			(show_name no)
@@
 			(project "CycleSync"
 				(path "/3f2cc6af-e67b-48ad-b391-ff7619611bd8/b5b9e253-8b7f-4bb9-bef8-83286ffed738"
-					(reference "R24")
+					(reference "R25")
 					(unit 1)
 				)
@@
 		(dnp no)
 		(fields_autoplaced yes)
-		(property "Reference" "C35"
+		(property "Reference" "C36"
 			(at 226.06 86.3599 0)
 			(show_name no)
@@
 			(project "CycleSync"
 				(path "/3f2cc6af-e67b-48ad-b391-ff7619611bd8/b5b9e253-8b7f-4bb9-bef8-83286ffed738"
-					(reference "C35")
+					(reference "C36")
 					(unit 1)
 				)
@@
 		(dnp no)
 		(fields_autoplaced yes)
-		(property "Reference" "C36"
+		(property "Reference" "C37"
 			(at 236.22 76.2 90)
 			(show_name no)
@@
 			(project "CycleSync"
 				(path "/3f2cc6af-e67b-48ad-b391-ff7619611bd8/b5b9e253-8b7f-4bb9-bef8-83286ffed738"
-					(reference "C36")
+					(reference "C37")
 					(unit 1)
 				)
@@
 		(dnp no)
 		(fields_autoplaced yes)
-		(property "Reference" "C31"
+		(property "Reference" "C32"
 			(at 151.13 110.4899 0)
 			(show_name no)
@@
 			(project "CycleSync"
 				(path "/3f2cc6af-e67b-48ad-b391-ff7619611bd8/b5b9e253-8b7f-4bb9-bef8-83286ffed738"
-					(reference "C31")
+					(reference "C32")
 					(unit 1)
 				)
@@
 		(dnp no)
 		(fields_autoplaced yes)
-		(property "Reference" "C27"
+		(property "Reference" "C28"
 			(at 106.68 74.9299 0)
 			(show_name no)
@@
 			(project "CycleSync"
 				(path "/3f2cc6af-e67b-48ad-b391-ff7619611bd8/b5b9e253-8b7f-4bb9-bef8-83286ffed738"
-					(reference "C27")
+					(reference "C28")
 					(unit 1)
 				)
@@
 		(in_pos_files yes)
 		(dnp no)
-		(property "Reference" "U4"
+		(property "Reference" "U5"
 			(at 131.572 96.52 0)
 			(show_name no)
@@
 			(project "CycleSync"
 				(path "/3f2cc6af-e67b-48ad-b391-ff7619611bd8/b5b9e253-8b7f-4bb9-bef8-83286ffed738"
-					(reference "U4")
+					(reference "U5")
 					(unit 1)
 				)
@@
 		(in_pos_files yes)
 		(dnp no)
-		(property "Reference" "C34"
+		(property "Reference" "C35"
 			(at 186.944 123.952 0)
 			(show_name no)
@@
 			(project "CycleSync"
 				(path "/3f2cc6af-e67b-48ad-b391-ff7619611bd8/b5b9e253-8b7f-4bb9-bef8-83286ffed738"
-					(reference "C34")
+					(reference "C35")
 					(unit 1)
 				)
@@
 		(dnp no)
 		(fields_autoplaced yes)
-		(property "Reference" "C30"
+		(property "Reference" "C31"
 			(at 153.67 71.1199 0)
 			(show_name no)
@@
 			(project "CycleSync"
 				(path "/3f2cc6af-e67b-48ad-b391-ff7619611bd8/b5b9e253-8b7f-4bb9-bef8-83286ffed738"
-					(reference "C30")
+					(reference "C31")
 					(unit 1)
 				)
@@
 		(dnp no)
 		(fields_autoplaced yes)
-		(property "Reference" "C28"
+		(property "Reference" "C29"
 			(at 116.84 74.9299 0)
 			(show_name no)
@@
 			(project "CycleSync"
 				(path "/3f2cc6af-e67b-48ad-b391-ff7619611bd8/b5b9e253-8b7f-4bb9-bef8-83286ffed738"
-					(reference "C28")
+					(reference "C29")
 					(unit 1)
 				)
