File: CycleSync/Daughter_IO.kicad_sch (KiCad schematic)
At the start: 17 parts, among them J3 USB4085-GF-A, J4 STX-3501-3N, J5 STX-3501-3N, J6 5499923-1, J7 5499923-4, J8 USB4085-GF-A, U14 TPD2EUSB30A, U15 TPD2EUSB30ADRTR, U16 TPD2E2U06DCKR, U17 TPD2E2U06DCKR

Commit message: verified schematic wirings
Parts:
- added R56, R57: 10k, symbol Device:R
- renumbered D9 to D10, D5 to D11, D6 to D7, D7 to D8, D10 to D9, J8 to J4, J4 to J8, R51 to R54, R52 to R55, U14 to U18, U15 to U19, U16 to U20
Connections:
- net LINE_IN_L: now also R57.2; no longer J5.T
- net LINE_IN_R: now also R56.2; no longer J5.R
- new net: J5.R, R56.1
- new net: J5.T, R57.1
Other:
- note added: "HOST USB-C: USB 2.0 DATA & VBUS"
- note added: "J4 IS A USB-C 5 V POWER INPUT ONLY. R41/R42 PRESENT Rd ON CC1/CC2. NO USB DATA AND NO HIGHER-VOLTAGE 9/12/15/20 V PD NEGOTIATION ON J4."
- note added: "USB-C 5 V POWER INPUT"
- note removed: "HOST USB-C — USB 2.0 DATA & VBUS"
- note removed: "PD USB-C — POWER INPUT ONLY"

Commit message: added some new testpoints for I2C
Parts:
- D10, D9: footprint Package_TO_SOT_SMD:SOT-523 -> Diode_SMD:D_SOD-523
- R54, R55, R56, R57: footprint (none) -> Resistor_SMD:R_0603_1608Metric
- renumbered U17 to U16, U18 to U17, U19 to U18, U20 to U19
Changed lines of the file:
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@@
 			)
 		)
-		(property "Footprint" ""
+		(property "Footprint" "Resistor_SMD:R_0603_1608Metric"
 			(at 38.1 30.988 90)
 			(hide yes)
@@
 		(dnp no)
 		(fields_autoplaced yes)
-		(property "Reference" "U20"
+		(property "Reference" "U19"
 			(at 236.22 118.11 0)
 			(show_name no)
@@
 			)
 		)
-		(property "Datasheet" "http://www.ti.com/lit/ds/symlink/tpd2eusb30a.pdf"
+		(property "Datasheet" "https://www.ti.com/lit/ds/symlink/tpd2e2u06.pdf"
 			(at 236.22 128.27 0)
 			(hide yes)
@@
 			(project "CycleSync"
 				(path "/3f2cc6af-e67b-48ad-b391-ff7619611bd8/afe1aeae-2b35-4a9c-80c8-33387c6b1d4e"
-					(reference "U20")
+					(reference "U19")
 					(unit 1)
 				)
@@
 			)
 		)
-		(property "Footprint" "Package_TO_SOT_SMD:SOT-523"
+		(property "Footprint" "Diode_SMD:D_SOD-523"
 			(at 256.54 99.06 0)
 			(hide yes)
@@
 		(dnp no)
 		(fields_autoplaced yes)
-		(property "Reference" "U19"
+		(property "Reference" "U18"
 			(at 270.51 38.1 0)
 			(show_name no)
@@
 			(project "CycleSync"
 				(path "/3f2cc6af-e67b-48ad-b391-ff7619611bd8/afe1aeae-2b35-4a9c-80c8-33387c6b1d4e"
-					(reference "U19")
+					(reference "U18")
 					(unit 1)
 				)
@@
 			)
 		)
-		(property "Footprint" ""
+		(property "Footprint" "Resistor_SMD:R_0603_1608Metric"
 			(at 101.6 28.448 90)
 			(hide yes)
@@
 			)
 		)
-		(property "Footprint" "Package_TO_SOT_SMD:SOT-523"
+		(property "Footprint" "Diode_SMD:D_SOD-523"
 			(at 53.34 66.04 0)
 			(hide yes)
@@
 			)
 		)
-		(property "Footprint" ""
+		(property "Footprint" "Resistor_SMD:R_0603_1608Metric"
 			(at 40.64 178.308 90)
 			(hide yes)
@@
 			)
 		)
-		(property "Footprint" ""
+		(property "Footprint" "Resistor_SMD:R_0603_1608Metric"
 			(at 46.99 193.548 90)
 			(hide yes)
@@
 		(dnp no)
 		(fields_autoplaced yes)
-		(property "Reference" "U17"
+		(property "Reference" "U16"
 			(at 85.09 60.96 0)
 			(show_name no)
@@
 			)
 		)
-		(property "Datasheet" "http://www.ti.com/lit/ds/symlink/tpd2eusb30a.pdf"
+		(property "Datasheet" "https://www.ti.com/lit/ds/symlink/tpd2e2u06.pdf"
 			(at 85.09 71.12 0)
 			(hide yes)
@@
 			(project "CycleSync"
 				(path "/3f2cc6af-e67b-48ad-b391-ff7619611bd8/afe1aeae-2b35-4a9c-80c8-33387c6b1d4e"
-					(reference "U17")
+					(reference "U16")
 					(unit 1)
 				)
@@
 		(in_pos_files yes)
 		(dnp no)
-		(property "Reference" "U18"
+		(property "Reference" "U17"
 			(at 74.93 107.696 0)
 			(show_name no)
@@
 			(project "CycleSync"
 				(path "/3f2cc6af-e67b-48ad-b391-ff7619611bd8/afe1aeae-2b35-4a9c-80c8-33387c6b1d4e"
-					(reference "U18")
-					(unit 1)
-				)
+					(reference "U17")
+					(unit 1)
+				)

Commit message: added footprints and manufacturer part number
Parts:
- D10, D9: Distributor Link (none) -> https://jlcpcb.com/partdetail/TexasInstruments-TPD1E10B06DY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; MANUFACTURER (none) -> Texas Instruments; MPN (none) -> TPD1E10B06DYAR
- D11: Distributor Link (none) -> https://jlcpcb.com/partdetail/TexasInstruments-ESD2CAN24DBZ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; MANUFACTURER (none) -> Texas Instruments; MPN (none) -> ESD2CAN24DBZRQ1
- D7, D8: Distributor Link (none) -> https://jlcpcb.com/partdetail/Kingbright-KP1608MGC/C598258; MANUFACTURER (none) -> Kingbright; MPN (none) -> KP-1608MGC
- J3, J4: footprint (none) -> USB4085-GF-A_REVB:GCT_USB4085-GF-A_REVB; Distributor Link (none) -> https://jlcpcb.com/partdetail/8061907-USB4085_GFA/C7095263; MANUFACTURER (none) -> Global Connector Technology; MPN (none) -> USB4085-GF-A
- J5: footprint (none) -> STX-3501-3N:STX35013N; Distributor Link (none) -> https://www.digikey.com/en/products/detail/kycon-inc/STX-35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; MANUFACTURER (none) -> Kycon; MPN (none) -> STX-3501-3N; Notes (none) -> It is out of stock in JLCPCB
- J6: footprint (none) -> 5499923-1:TE_5499923-1; Distributor Link (none) -> https://www.digikey.com/en/products/detail/te-connectivity-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; MANUFACTURER (none) -> TE Connectivity AMP Connectors; MPN (none) -> 5499923-1; Notes (none) -> It is out of stock in JLCPCB
- J7: footprint (none) -> 5499923-4:TE_5499923-4; Distributor Link (none) -> https://www.digikey.com/en/products/detail/te-connectivity-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; MANUFACTURER (none) -> TE Connectivity AMP Connectors; MPN (none) -> 5499923-4; Notes (none) -> It is out of stock in JLCPCB
- J8: footprint (none) -> STX-3501-3N:STX35013N; Distributor Link (none) -> https://www.digikey.com/en/products/detail/kycon-inc/STX-35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; MANUFACTURER (none) -> Kycon, Inc.; MPN (none) -> STX-3501-3N; Notes (none) -> It is out of stock in JLCPCB
- R54: Distributor Link (none) -> https://jlcpcb.com/partdetail/25994-0603WAJ0621T5E/C25251; MANUFACTURER (none) -> UNI-ROYAL(Uniroyal Elec); MPN (none) -> 0603WAJ0621T5E
- R55: Distributor Link (none) -> https://jlcpcb.com/partdetail/23878-0603WAF3900T5E/C23151; MANUFACTURER (none) -> UNI-ROYAL(Uniroyal Elec); MPN (none) -> 0603WAF3900T5E
- R56, R57: Distributor Link (none) -> https://jlcpcb.com/partdetail/YAGEO-RC0603FR0710KL/C98220; MANUFACTURER (none) -> YAGEO; MPN (none) -> RC0603FR-0710KL
- U16, U19: Distributor Link (none) -> https://jlcpcb.com/partdetail/TexasInstruments-TPD2E2U06DCK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; MANUFACTURER (none) -> Texas Instruments; MPN (none) -> TPD2E2U06DCKR
- U17: value TPD2EUSB30A -> TPD2EUSB30ADRTR; Distributor Link (none) -> https://jlcpcb.com/partdetail/TexasInstruments-TPD2EUSB30AD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; MANUFACTURER (none) -> Texas Instruments; MPN (none) -> TPD2EUSB30ADRTR
- U18: Distributor Link (none) -> https://jlcpcb.com/partdetail/TexasInstruments-TPD2EUSB30AD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; MANUFACTURER (none) -> Texas Instruments; MPN (none) -> TPD2EUSB30ADRTR
