File: CycleSync/GNSS_RF.kicad_sch (KiCad schematic)
At the start: 1 part, among them U2 LC76G

Commit message: finished Phase 1.4
Parts:
- added ANT1: YFGC035WWB, symbol Device:Antenna
- added BT1: Battery_Cell, symbol Device:Battery_Cell
- added C10, C15: 33p, symbol Device:C
- added C11, C16: 100n, symbol Device:C
- added C12: 4u7, symbol Device:C
- added C13, C14: C, symbol Device:C
- added C17: 10u, symbol Device:C
- added D1, D2, D3: D_TVS, symbol Device:D_TVS
- added FL1: SAFFA1G58KA0F0A, Filter:Filter_1411-5_1.4x1.1mm, symbol Filter:SAFFA1G58KA0F0A
- added J2: UFL_NM_shares_pad_w_R13, symbol Connector:Conn_Coaxial
- added L1, L2: L, symbol Device:L
- added R10, R9: R, symbol Device:R
- added R11: 10k, symbol Device:R
- added R12, R13, R6, R7, R8: 0R, symbol Device:R
- added R5: 1k, symbol Device:R
Connections:
- net GND is gone; now on net +3.3V: U2.1 (GND), U2.10 (GND), U2.12 (GND), U2.28 (GND)
- net GNSS_RESET_N: now also R12.1; no longer U2.9 (~{RESET})
- net at U2.11 (RF_IN): now also R10.1, R6.2
- net at U2.24 (D_SEL): now also R11.2
- net at U2.6 (V_BCKP): now also BT1.1 (+), C10.1, C11.1, C12.1, D1.2 (A2), R5.1
- net +3.3V: now reaches U2.8 (VCC)
- net +3.3V: now also BT1.2 (-), C10.2, C11.2, C12.2, C13.2, C14.2, C15.1, C15.2, C16.1, C16.2, C17.1, C17.2, D1.1 (A1), D2.1 (A1), D3.1 (A1), D3.2 (A2), FL1.2, FL1.3, FL1.5, J2.2 (Ext), L1.2, L2.2, R11.1, R5.2
- new net: J2.1 (In), R13.2, R7.1, R9.1
- new net: ANT1.1 (A), C13.1, D2.2 (A2), R8.1
- new net: C14.1, R13.1, R8.2
- new net: R6.1, R7.2
- new net: FL1.4, L2.1, R10.2
- new net: FL1.1, L1.1, R9.2
- new net: R12.2, U2.9 (~{RESET})
- no-connect marks 0 -> 10

Commit message: s
Parts:
- removed C10: 33p, symbol Device:C
- removed C11: 100n, symbol Device:C
- removed C12: 4u7, symbol Device:C
- removed R5: 1k, symbol Device:R
- added C21: 33p, symbol Device:C
- added C22: 100n, symbol Device:C
- added C23: 4u7, symbol Device:C
- added C24, C83: 1u, symbol Device:C
- added Q1: 2N7002, Package_TO_SOT_SMD:SOT-23, symbol Transistor_FET:2N7002
- added R15: 1k, symbol Device:R
- added R16, R18: 100k, symbol Device:R
- added R17: 10k, symbol Device:R
- added R19, R20, R21, R22: 0R, symbol Device:R
- added TP10, TP11, TP15, TP5, TP6, TP7, TP8, TP9: TestPoint, symbol Connector:TestPoint
- added U13: TPS22919DCK, Package_TO_SOT_SMD:SOT-363_SC-70-6, symbol Power_Management:TPS22919DCK
- added U18: MAX40203AUK+T, Package_TO_SOT_SMD:SOT-23-5, symbol CycleSync_local:MAX40203AUK
- BT1: value Battery_Cell -> VL-2330/HFN
- C16: renamed from C13; value C -> NM; now not fitted
- C17: renamed from C14; value C -> NM; now not fitted
- D1: value D_TVS -> TPD1E1B04DPYR; footprint (none) -> Diode_SMD:D_0402_1005Metric
- D2, D3: value D_TVS -> TPD1E0B04DPYR
- FL1: value SAFFA1G58KA0F0A -> B39162B2618P810; footprint Filter:Filter_1411-5_1.4x1.1mm -> Filter:Filter_1109-5_1.1x0.9mm
- J2: value UFL_NM_shares_pad_w_R13 -> U.FL-R-SMT-1(10); footprint (none) -> Connector_Coaxial:U.FL_Hirose_U.FL-R-SMT-1_Vertical
- L1, L2: value L -> NM; now not fitted
- R11: renamed from R9; value R -> NM; now not fitted
- R12: renamed from R10; value R -> NM; now not fitted
- renumbered C15 to C18, C16 to C19, C17 to C20, R6 to R10, R11 to R13, R12 to R14, R8 to R7, R13 to R8, R7 to R9
Connections:
- net PPS_IN: now also R19.2, TP15.1; no longer U2.4 (1PPS)
- net UART_RX: now also R21.2; no longer U2.2 (TXD)
- net UART_TX: now also R22.2; no longer U2.3 (RXD)
- net RF_POST_TP: now reaches R11.1, R8.2, R9.1
- net RF_POST_TP: no longer J2.1 (In)
- net RF_ANT: now reaches ANT1.1 (A), C16.1, D2.2 (A2), R7.1
- net RF_MATCHED: now reaches C17.1, R7.2, R8.1
- net RF_MATCHED: now also J2.1 (In)
- net D_SEL: now reaches R13.2, U2.24 (D_SEL)
- net RF_FILTERED: now reaches R10.1, R9.2
- net V_BCKP: now reaches D1.2 (A2), U2.6 (V_BCKP)
- net V_BCKP: now also C21.1, C22.1, C23.1, TP9.1, U13.5 (QOD), U13.6 (OUT); no longer BT1.1 (+)
- net RF_IN: now reaches R10.2, R12.1, U2.11 (RF_IN)
- net RESET_MODULE_N: now reaches R14.2, U2.9 (~{RESET})
- net RESET_MODULE_N: now also TP8.1
- net +3.3V renamed GND
- net GND: now also C21.2, C22.2, C23.2, C24.2, C83.2, Q1.2 (S), R18.1, TP10.1, U13.2 (GND), U18.2 (GND); no longer C18.1, C19.1, C20.1, D3.2 (A2), R13.1, U2.8 (VCC)
- net GNSS_FIX renamed 3D_FIX
- net 3D_FIX: now also R20.1
- new net +3V3_GNSS: C18.1, C19.1, C20.1, C83.1, D3.2 (A2), R13.1, TP7.1, U18.1 (VDD), U18.3 (EN), U2.8 (VCC)
- new net 1PPS: R19.1, U2.4 (1PPS)
- new net BCKP_CELL: BT1.1 (+), R15.1, R16.2, TP11.1, U13.1 (IN)
- new net BCKP_CHG: C24.1, R15.2, U18.5 (OUT)
- new net BCKP_GATE: Q1.1 (G), R17.2, R18.2
- new net BCKP_SW_EN: Q1.3 (D), R16.1, U13.3 (ON)
- new net GNSS_BCKP_CUTOFF: R17.1
- new net GNSS_FIX_STATUS: R20.2
- new net RXD: R22.1, TP6.1, U2.3 (RXD)
- new net TXD: R21.1, TP5.1, U2.2 (TXD)
Other:
- note added: "BACKUP-DOMAIN NOTES BT1 MUST BE A RECHARGEABLE VL-2330/HFN CELL. DO NOT SUBSTITUTE A PRIMARY COIN CELL. R15 = 1 kΩ LIMITS THE CELL CHARGE CURRENT. V_BCKP MUST RISE BEFORE OR WITH U2 VCC. U13 QOD IS INTENTIONALLY CONNECTED TO OUT. U18 BLOCKS BT1 BACKFEED INTO +3V3_GNSS WHEN GNSS POWER IS OFF."
- note added: "GNSS ANTENNA & 50 Ω RF FRONT END"
- note added: "GNSS RESET: R14 = 0 Ω, POPULATE D_SEL STRAP: R13 = DNP FOR UART DEFAULT"
- note added: "LC76G GNSS MODULE & INTERFACES"
- note added: "RF POPULATION OPTIONS DEFAULT: FIT R7-R10 = 0 Ω. DNP C16, C17, R11, R12, L1, L2, J2, FL1. VNA TEST: DNP R8; FIT J2. SAW FILTER: DNP R9 AND R10; FIT FL1 AND R11/R12 = 0 Ω. KEEP L1/L2 DNP."
- note added: "V_BCKP BACKUP DOMAIN & CUTOFF"
- title: (none) -> LC76G GNSS, RF FRONT END & BACKUP DOMAIN
- moved on the sheet: ANT1, C18, C19, C20, D2, D3, FL1, J2, R10, R13, R14, R7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

Commit message: verified schematic wirings
Parts:
- renumbered C83 to C21, C24 to C22, C21 to C23, C22 to C24, C23 to C25, R13 to R10, R7 to R11, R8 to R12, R9 to R13, R10 to R14, R11 to R15, R12 to R16, R19 to R17, R20 to R18, R21 to R19, R22 to R20, R15 to R21, R16 to R22, R17 to R23, R18 to R24, R14 to R9, U18 to U3, U13 to U4
Other:
- note added: "BACKUP-DOMAIN NOTES BT1 MUST BE A RECHARGEABLE VL-2330/HFN CELL. DO NOT SUBSTITUTE A PRIMARY COIN CELL. R21 = 1 kΩ LIMITS CELL CHARGE CURRENT. U3 BLOCKS BT1 BACKFEED INTO +3V3_GNSS. U4 QOD IS INTENTIONALLY CONNECTED TO OUT. V_BCKP MUST RISE BEFORE OR WITH U2 VCC. GPIO12 HIGH = BACKUP OFF. GPIO12 LOW OR HI-Z = BACKUP ON."
- note added: "GNSS RESET: R9 = 0 Ω, POPULATE D_SEL STRAP: R10 = DNP FOR UART DEFAULT"
- note added: "RF POPULATION OPTIONS DEFAULT: FIT R11-R14 = 0 Ω. DNP C16, C17, R15, R16, L1, L2, J2, FL1. VNA TEST: DNP R12; FIT J2. SAW FILTER: DNP R13 AND R14. FIT FL1 AND FIT R15/R16 = 0 Ω. KEEP L1/L2 DNP."
- note removed: "BACKUP-DOMAIN NOTES BT1 MUST BE A RECHARGEABLE VL-2330/HFN CELL. DO NOT SUBSTITUTE A PRIMARY COIN CELL. R15 = 1 kΩ LIMITS THE CELL CHARGE CURRENT. V_BCKP MUST RISE BEFORE OR WITH U2 VCC. U13 QOD IS INTENTIONALLY CONNECTED TO OUT. U18 BLOCKS BT1 BACKFEED INTO +3V3_GNSS WHEN GNSS POWER IS OFF."
- note removed: "GNSS RESET: R14 = 0 Ω, POPULATE D_SEL STRAP: R13 = DNP FOR UART DEFAULT"
- note removed: "RF POPULATION OPTIONS DEFAULT: FIT R7-R10 = 0 Ω. DNP C16, C17, R11, R12, L1, L2, J2, FL1. VNA TEST: DNP R8; FIT J2. SAW FILTER: DNP R9 AND R10; FIT FL1 AND R11/R12 = 0 Ω. KEEP L1/L2 DNP."
- moved on the sheet: C22

Commit message: added some new testpoints for I2C
Parts:
- C16, C17, C18, C19, C23, C24: footprint (none) -> Capacitor_SMD:C_0402_1005Metric
- C20, C25: footprint (none) -> Capacitor_SMD:C_0805_2012Metric
- C21, C22: footprint (none) -> Capacitor_SMD:C_0603_1608Metric
- D1: footprint Diode_SMD:D_0402_1005Metric -> Diode_SMD:D_SOD-523
- D2, D3: footprint (none) -> Diode_SMD:D_SOD-882
- R10, R11, R12, R13, R14, R15, R16, R17, R18, R19, R20, R21, R22, R23, R24, R9: footprint (none) -> Resistor_SMD:R_0402_1005Metric
- TP10: renamed from TP11; value TestPoint -> V_BCKP_CHG; footprint (none) -> TestPoint:TestPoint_Pad_D1.5mm
- TP3: renamed from TP8; value TestPoint -> GNSS_RESET_N; footprint (none) -> TestPoint:TestPoint_Pad_D1.5mm
- TP4: renamed from TP7; value TestPoint -> +3V3_GNSS; footprint (none) -> TestPoint:TestPoint_Pad_D1.5mm
- TP5: renamed from TP15; value TestPoint -> PPS_IN; footprint (none) -> TestPoint:TestPoint_Pad_D1.5mm
- TP6: renamed from TP5; value TestPoint -> UART_RX; footprint (none) -> TestPoint:TestPoint_Pad_D1.5mm
- TP7: renamed from TP6; value TestPoint -> UART_TX; footprint (none) -> TestPoint:TestPoint_Pad_D1.5mm
- TP8: renamed from TP10; value TestPoint -> GND; footprint (none) -> TestPoint:TestPoint_Pad_D1.5mm
- TP9: value TestPoint -> V_BCKP; footprint (none) -> TestPoint:TestPoint_Pad_D1.5mm
Other:
- moved on the sheet: TP3

Commit message: added footprints and manufacturer part number
Parts:
- ANT1: footprint (none) -> YFGC035WWB:XDCR_YFGC035WWB; Distributor Link (none) -> https://www.digikey.com/en/products/detail/quectel/YFGC035W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; MANUFACTURER (none) -> Quectel; MPN (none) -> YFGC035WWB; Notes (none) -> It is out of stock in JLCPCB
- BT1: footprint (none) -> VL_2330_HFN:VL2330HFN; Distributor Link (none) -> https://www.digikey.com/en/products/detail/panasonic-energy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; MANUFACTURER (none) -> Panasonic Energy; MPN (none) -> VL-2330/HFN; Notes (none) -> It is out of stock in JLCPCB
- C18, C23: Distributor Link (none) -> https://jlcpcb.com/partdetail/137786-GCM1555C1H330JA16D/C12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; MANUFACTURER (none) -> Murata Electronics; MPN (none) -> GCM1555C1H330JA16D
- C19, C24: Distributor Link (none) -> https://jlcpcb.com/partdetail/MurataElectronics-GRM155R71A1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; MANUFACTURER (none) -> Murata Electronics; MPN (none) -> GRM155R71A104KA01D
- C20: Distributor Link (none) -> https://jlcpcb.com/partdetail/236937-GRM21BZ71E106KE15L/C23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; MANUFACTURER (none) -> Murata Electronics; MPN (none) -> GRM21BZ71E106KE15L
- C21, C22: Distributor Link (none) -> https://jlcpcb.com/partdetail/30690-CL10B105KA8NNNC/C29936; MANUFACTURER (none) -> Samsung Electro-Mechanics; MPN (none) -> CL10B105KA8NNNC
- C25: Distributor Link (none) -> https://jlcpcb.com/partdetail/2131-CL21A475KAQNNNE/C1779; MANUFACTURER (none) -> Samsung Electro-Mechanics; MPN (none) -> CL21A475KAQNNNE
- D1: value TPD1E1B04DPYR -> TPD1E0B04DPYR; footprint Diode_SMD:D_SOD-523 -> Diode_SMD:D_SOD-882; Distributor Link (none) -> https://jlcpcb.com/partdetail/TexasInstruments-TPD1E0B04DPY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; MANUFACTURER (none) -> Texas Instruments; MPN (none) -> TPD1E0B04DPYR
- D2, D3: Distributor Link (none) -> https://jlcpcb.com/partdetail/TexasInstruments-TPD1E0B04DPY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; MANUFACTURER (none) -> Texas Instruments; MPN (none) -> TPD1E0B04DPYR
- FL1: Distributor Link (none) -> https://jlcpcb.com/partdetail/Qualcomm-B39162B2618P810/C328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; MANUFACTURER (none) -> Qualcomm; MPN (none) -> B39162B2618P810
- J2: Distributor Link (none) -> https://jlcpcb.com/partdetail/HRS_Hirose-U_FL_R_SMT_1_10/C8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; MANUFACTURER (none) -> HRS(Hirose); MPN (none) -> U.FL-R-SMT-1(10)
- L1, L2: footprint (none) -> Inductor_SMD:L_0402_1005Metric
- Q1: Distributor Link (none) -> https://jlcpcb.com/partdetail/JSCJ-2N7002/C8545; MANUFACTURER (none) -> Jiangsu Changjing Electronics Technology Co., Ltd.; MPN (none) -> 2N7002
- R10, R23: Distributor Link (none) -> https://jlcpcb.com/partdetail/YAGEO-RC0402FR0710KL/C60490; MANUFACTURER (none) -> YAGEO; MPN (none) -> RC0402FR-0710KL
- R11, R12, R13, R14, R17, R18, R19, R20, R9: Distributor Link (none) -> https://jlcpcb.com/partdetail/YAGEO-RC0402FR070RL/C106231; MANUFACTURER (none) -> YAGEO; MPN (none) -> RC0402FR-070RL
- R21: Distributor Link (none) -> https://jlcpcb.com/partdetail/VishayIntertech-CRCW04021K00F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; MANUFACTURER (none) -> Vishay Intertech; MPN (none) -> CRCW04021K00FKED
- R22, R24: Distributor Link (none) -> https://jlcpcb.com/partdetail/YAGEO-RC0402FR07100KL/C60491; MANUFACTURER (none) -> YAGEO; MPN (none) -> RC0402FR-07100KL
- TP10, TP3, TP4, TP5, TP6, TP7, TP9: now left out of the parts list
- TP8: value GND -> GND_RF; now left out of the parts list
- U2: value LC76G -> LC76GAB; Distributor Link (none) -> https://jlcpcb.com/partdetail/Quectel-LC76GABMD/C7437114; MPN (none) -> LC76GABMD
- U3: Distributor Link (none) -> https://jlcpcb.com/partdetail/2745548-MAX40203AUKT/C2653639; MANUFACTURER (none) -> Analog Devices Inc./Maxim Integrated; MPN (none) -> MAX40203AUK+T
- U4: value TPS22919DCK -> TPS22919DCKR; Distributor Link (none) -> https://jlcpcb.com/partdetail/TexasInstruments-TPS22919DCKR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; MANUFACTURER (none) -> Texas Instruments; MPN (none) -> TPS22919DCKR
