File: CycleSync/USB_PD.kicad_sch (KiCad schematic)
At the start: 0 parts

Commit message: finishing Phase 1.5
Parts:
- added R28, R30, R31, R32: 2.2k, symbol Device:R
- added R29, R33: 10k, symbol Device:R
- added U5: TPS25751D, CycleSync_local:REF0038A_TPS25751D, symbol CycleSync_local:TPS25751D
Connections:
- net I2C_SCL: now also R28.1, U5.9 (I2Ct_SCL)
- net I2C_SDA: now also R30.1, U5.8 (I2Ct_SDA)
- new net: R32.1, U5.16 (I2Cc_SDA)
- new net: R31.1, U5.17 (I2Cc_SCL)
- new net: U5.15 (DRAIN), U5.30 (DRAIN)
- new net: R33.1, U5.18 (I2Cc_IRQ)
- new net: U5.20 (PPHV), U5.21 (PPHV), U5.22 (PPHV)
- new net: U5.23 (VBUS_IN), U5.24 (VBUS_IN), U5.25 (VBUS_IN)
- new net: U5.32 (VBUS), U5.33 (VBUS)
- new net GND: U5.11 (GND), U5.12 (GND), U5.14 (GND), U5.31 (GND)
- new net LDO_3V3: R28.2, R29.2, R30.2, R31.2, R32.2, R33.2, U5.1 (LDO_3v3)
- new net PD_IRQ: R29.1, U5.10 (I2Ct_IRQ)
- new net PP5V: U5.34 (PP5V), U5.35 (PP5V)

Commit message: s
Parts:
- removed R28, R30: 2.2k, symbol Device:R
- removed R29: 10k, symbol Device:R
- added C50: 100n, symbol Device:C
- added C51, C52, C53, C66, C67: 10u, symbol Device:C
- added C54, C55: 22u, symbol Device:C
- added C56: 0u1, symbol Device:C
- added C57, C58: 330p, Capacitor_SMD:C_0402_1005Metric, symbol Device:C
- added C59, C60, C61, C62: 0u01, symbol Device:C
- added C63: 4u7, symbol Device:C
- added C64, C65: 100u, symbol Device:C
- added R34, R35, R37, R38: 2k2, symbol Device:R
- added R36: 10k, symbol Device:R
- added R39, R40: 0R, symbol Device:R
- added R41, R42: 5.1k, Resistor_SMD:R_0402_1005Metric, symbol Device:R
- added TP1: EEPROM_SDA, symbol Connector:TestPoint
- added TP2: EEPROM_SCL, symbol Connector:TestPoint
- added TP3: EEPROM_3V3, symbol Connector:TestPoint
- added TP4: EEPROM_GND, symbol Connector:TestPoint
- added U6: CAT24C512WI-GT3, Package_SO:SOIC-8_3.9x4.9mm_P1.27mm, symbol CycleSync_local:CAT24C512
- added U7: TVS2200DRV, Package_SON:WSON-6-1EP_2x2mm_P0.65mm_EP1x1.6mm, symbol Power_Protection:TVS2200DRV
- R31, R32: value 2.2k -> 5.1k; Variant (none) -> PD_OPTION
- R33, U5: Variant (none) -> PD_OPTION
Connections:
- net GND: now also R31.1, R32.1, U5.13 (GPIO11), U5.19 (GPIO3), U5.26 (GPIO4), U5.27 (GPIO5), U5.36 (GPIO7), U5.37 (GPIO6), U5.39 (GND), U5.5 (GPIO0), U5.6 (GPIO1), U5.7 (GPIO2), C50.2, C51.2, C52.2, C53.2, C54.2, C55.2, C56.2, C57.2, C58.2, C59.2, C60.2, C61.2, C62.2, C63.2, C64.2, C65.2, C66.2, C67.2, R39.1, R40.1, R41.2, R42.2, TP4.1, U6.1 (A0), U6.2 (A1), U6.3 (A2), U6.4 (GND), U6.7 (WP), U7.1 (GND), U7.2 (GND), U7.3 (GND), U7.7 (GND)
- net I2C_SCL: now also R38.1
- net I2C_SDA: now also R37.1
- net LDO_3V3: now also C50.1, C51.1, R34.2, R35.2, R36.2, R37.2, R38.2, TP3.1, U6.8 (VCC); no longer R31.2, R32.2
- net PD_IRQ: now also R36.1
- net PP5V: now also C64.1, C65.1, C66.1, C67.1
- net PD_EEPROM_SDA: now reaches U5.16 (I2Cc_SDA)
- net PD_EEPROM_SDA: now also R34.1, TP1.1, U6.5 (SDA); no longer R32.1
- net PD_EEPROM_SCL: now reaches U5.17 (I2Cc_SCL)
- net PD_EEPROM_SCL: now also R35.1, TP2.1, U6.6 (SCL); no longer R31.1
- net DRAIN: now reaches U5.15 (DRAIN), U5.30 (DRAIN)
- net DRAIN: now also U5.40 (DRAIN)
- net PD_I2CC_IRQ_N: now reaches R33.1, U5.18 (I2Cc_IRQ)
- net at U5.2 (ADCIN1): now also R40.2
- net PPHV: now reaches U5.20 (PPHV), U5.21 (PPHV), U5.22 (PPHV)
- net PPHV: now also C54.1, C55.1, C56.1
- net VBUS: now reaches U5.23 (VBUS_IN), U5.24 (VBUS_IN), U5.25 (VBUS_IN)
- net VBUS: now also U5.32 (VBUS), U5.33 (VBUS), C59.1, C60.1, C61.1, C62.1, C63.1, U7.4 (IN), U7.5 (IN), U7.6 (IN)
- net CC1: now reaches U5.28 (CC1)
- net CC1: now also C58.1, R42.1
- net CC2: now reaches U5.29 (CC2)
- net CC2: now also C57.1, R41.1
- net at U5.3 (ADCIN2): now also R39.2
- net +3V3_DIG: now reaches U5.38 (VIN_3V3)
- net +3V3_DIG: now also C52.1
- net LDO_1V5: now reaches U5.4 (LDO_1V5)
- net LDO_1V5: now also C53.1
- new net PDIN_CC1: R31.2
- new net PDIN_CC2: R32.2
Other:
- note added: "ADCIN1 = 0, ADCIN2 = 0"
- note added: "CC1/CC2 — PD / NO-PD OPTION"
- note added: "EEPROM SELF-BOOT & RECOVERY INTERFACE"
- note added: "PD POWER DOMAINS & DECOUPLING"
- note added: "PD-OPTION I²C1 PULL-UPS R37/R38 = 2.2 kΩ TO U5 LDO_3V3 POPULATE ONLY IN PD BUILDS. NO-PD BUILDS USE R53/R54 ON MCU SHEET. NEVER POPULATE BOTH PULL-UP PAIRS."
- note added: "SAFEMODE, I²C ADDRESS 0x21"
- note added: "TPS25751D USB-C PD CONTROLLER & POWER PATH"
- note added: "USB-PD / NO-PD POPULATION OPTIONS PD BUILD: POPULATE ALL PD_OPTION COMPONENTS. DNP ALL NO_PD_OPTION COMPONENTS. NO-PD BUILD: DNP ALL PD_OPTION COMPONENTS. POPULATE ALL NO_PD_OPTION COMPONENTS. C57 AND C58 ARE COMMON: POPULATE IN BOTH BUILDS. USB D+/D− BYPASS U5 AND CONNECT DIRECTLY BETWEEN THE HOST USB-C PORT AND MCU."
- title: (none) -> TPS25751D USB-C POWER DELIVERY
- moved on the sheet: R33, U5

Commit message: verified schematic wirings
Parts:
- renumbered C50 to C51, C51 to C52, C52 to C53, C53 to C54, C54 to C55, C55 to C56, C56 to C57, C57 to C58, C58 to C59, C59 to C60, C60 to C61, C61 to C62, C62 to C63, C63 to C64, C64 to C65, C65 to C66, C66 to C67, C67 to C68, R40 to R33, R39 to R34, R33 to R35, R34 to R36, R35 to R37, R36 to R38, R37 to R39, R38 to R40, R31 to R41, R32 to R42, R41 to R43, R42 to R44, U6 to U7, U5 to U8, U7 to U9
Connections:
- net PPHV renamed VBUS_PD_5V
Other:
- note added: "PD-OPTION I²C1 PULL-UPS R39/R40 = 2.2 kΩ TO U8 LDO_3V3. POPULATE ONLY IN PD BUILDS. NO-PD BUILDS USE R7/R8 ON MCU SHEET. NEVER POPULATE BOTH PULL-UP PAIRS."
- note added: "USB-PD / NO-PD POPULATION OPTIONS PD BUILD: POPULATE ALL PD_OPTION COMPONENTS. DNP ALL NO_PD_OPTION COMPONENTS. NO-PD BUILD: DNP ALL PD_OPTION COMPONENTS. POPULATE ALL NO_PD_OPTION COMPONENTS. C58 AND C59 ARE COMMON: POPULATE IN BOTH BUILDS. USB D+/D− BYPASS U5 AND CONNECT DIRECTLY BETWEEN THE HOST USB-C PORT AND MCU."
- note removed: "PD-OPTION I²C1 PULL-UPS R37/R38 = 2.2 kΩ TO U5 LDO_3V3 POPULATE ONLY IN PD BUILDS. NO-PD BUILDS USE R53/R54 ON MCU SHEET. NEVER POPULATE BOTH PULL-UP PAIRS."
- note removed: "USB-PD / NO-PD POPULATION OPTIONS PD BUILD: POPULATE ALL PD_OPTION COMPONENTS. DNP ALL NO_PD_OPTION COMPONENTS. NO-PD BUILD: DNP ALL PD_OPTION COMPONENTS. POPULATE ALL NO_PD_OPTION COMPONENTS. C57 AND C58 ARE COMMON: POPULATE IN BOTH BUILDS. USB D+/D− BYPASS U5 AND CONNECT DIRECTLY BETWEEN THE HOST USB-C PORT AND MCU."
- moved on the sheet: R42

Commit message: added some new testpoints for I2C
Parts:
- C51, C57, C60, C61, C62, C63: footprint (none) -> Capacitor_SMD:C_0402_1005Metric
- C52, C53, C54, C64, C67, C68: footprint (none) -> Capacitor_SMD:C_0805_2012Metric
- C55, C56: footprint (none) -> Capacitor_SMD:C_1206_3216Metric
- C65, C66: footprint (none) -> Capacitor_SMD:C_1210_3225Metric
- R33, R34, R35, R36, R37, R38, R39, R40, R41, R42: footprint (none) -> Resistor_SMD:R_0402_1005Metric
- TP15: renamed from TP1; footprint (none) -> TestPoint:TestPoint_Pad_D2.0mm
- TP16: renamed from TP2; footprint (none) -> TestPoint:TestPoint_Pad_D2.0mm
- TP17: renamed from TP3; footprint (none) -> TestPoint:TestPoint_Pad_D2.0mm
- TP18: renamed from TP4; footprint (none) -> TestPoint:TestPoint_Pad_D2.0mm
Other:
- note added: "USB-PD / NO-PD POPULATION OPTIONS PD BUILD: POPULATE ALL PD_OPTION COMPONENTS. DNP ALL NO_PD_OPTION COMPONENTS. NO-PD BUILD: DNP ALL PD_OPTION COMPONENTS. POPULATE ALL NO_PD_OPTION COMPONENTS. C58 AND C59 ARE COMMON: POPULATE IN BOTH BUILDS. USB D+/D− BYPASS U8 AND CONNECT DIRECTLY BETWEEN THE HOST USB-C PORT AND MCU."
- note removed: "USB-PD / NO-PD POPULATION OPTIONS PD BUILD: POPULATE ALL PD_OPTION COMPONENTS. DNP ALL NO_PD_OPTION COMPONENTS. NO-PD BUILD: DNP ALL PD_OPTION COMPONENTS. POPULATE ALL NO_PD_OPTION COMPONENTS. C58 AND C59 ARE COMMON: POPULATE IN BOTH BUILDS. USB D+/D− BYPASS U5 AND CONNECT DIRECTLY BETWEEN THE HOST USB-C PORT AND MCU."
Changed lines of the file:
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@@
 		)
 	)
-	(text "USB-PD / NO-PD POPULATION OPTIONS\n\nPD BUILD:\nPOPULATE ALL PD_OPTION COMPONENTS.\nDNP ALL NO_PD_OPTION COMPONENTS.\n\nNO-PD BUILD:\nDNP ALL PD_OPTION COMPONENTS.\nPOPULATE ALL NO_PD_OPTION COMPONENTS.\n\nC58 AND C59 ARE COMMON:\nPOPULATE IN BOTH BUILDS.\n\nUSB D+/D− BYPASS U5 AND CONNECT DIRECTLY\nBETWEEN THE HOST USB-C PORT AND MCU."
+	(text "USB-PD / NO-PD POPULATION OPTIONS\n\nPD BUILD:\nPOPULATE ALL PD_OPTION COMPONENTS.\nDNP ALL NO_PD_OPTION COMPONENTS.\n\nNO-PD BUILD:\nDNP ALL PD_OPTION COMPONENTS.\nPOPULATE ALL NO_PD_OPTION COMPONENTS.\n\nC58 AND C59 ARE COMMON:\nPOPULATE IN BOTH BUILDS.\n\nUSB D+/D− BYPASS U8 AND CONNECT DIRECTLY\nBETWEEN THE HOST USB-C PORT AND MCU."
 		(exclude_from_sim no)
 		(at 188.976 149.352 0)
@@
 			)
 		)
-		(property "Footprint" ""
+		(property "Footprint" "Capacitor_SMD:C_1210_3225Metric"
 			(at 207.9752 121.92 0)
 			(hide yes)
@@
 			)
 		)
-		(property "Footprint" ""
+		(property "Footprint" "Resistor_SMD:R_0402_1005Metric"
 			(at 104.902 100.33 90)
 			(hide yes)
@@
 			)
 		)
-		(property "Footprint" ""
+		(property "Footprint" "Capacitor_SMD:C_0805_2012Metric"
 			(at 30.1752 166.37 0)
 			(hide yes)
@@
 			)
 		)
-		(property "Footprint" ""
+		(property "Footprint" "Capacitor_SMD:C_0402_1005Metric"
 			(at 232.1052 35.56 0)
 			(hide yes)
@@
 			)
 		)
-		(property "Footprint" ""
+		(property "Footprint" "Capacitor_SMD:C_0805_2012Metric"
 			(at 18.7452 166.37 0)
 			(hide yes)
@@
 			)
 		)
-		(property "Footprint" ""
+		(property "Footprint" "Capacitor_SMD:C_0402_1005Metric"
 			(at 220.6752 92.71 0)
 			(hide yes)
@@
 			)
 		)
-		(property "Footprint" ""
+		(property "Footprint" "Resistor_SMD:R_0402_1005Metric"
 			(at 96.012 100.33 90)
 			(hide yes)
@@
 			)
 		)
-		(property "Footprint" ""
+		(property "Footprint" "Capacitor_SMD:C_1206_3216Metric"
 			(at 206.7052 35.56 0)
 			(hide yes)
@@
 			)
 		)
-		(property "Footprint" ""
+		(property "Footprint" "Capacitor_SMD:C_0402_1005Metric"
 			(at 54.3052 64.77 0)
 			(hide yes)
@@
 			)
 		)
-		(property "Footprint" ""
+		(property "Footprint" "Resistor_SMD:R_0402_1005Metric"
 			(at 143.51 47.498 90)
 			(hide yes)
@@
 			)
 		)
-		(property "Footprint" ""
+		(property "Footprint" "Capacitor_SMD:C_1210_3225Metric"
 			(at 220.6752 121.92 0)
 			(hide yes)
@@
 			)
 		)
-		(property "Footprint" ""
+		(property "Footprint" "Resistor_SMD:R_0402_1005Metric"
 			(at 131.572 100.33 90)
 			(hide yes)
@@
 			)
 		)
-		(property "Footprint" ""
+		(property "Footprint" "Capacitor_SMD:C_0805_2012Metric"
 			(at 234.6452 121.92 0)
 			(hide yes)
@@
 			)
 		)
-		(property "Footprint" ""
+		(property "Footprint" "Capacitor_SMD:C_0402_1005Metric"
 			(at 232.1052 92.71 0)
 			(hide yes)
@@
 		(dnp no)
 		(fields_autoplaced yes)
-		(property "Reference" "TP2"
+		(property "Reference" "TP16"
 			(at 96.52 57.023 0)
 			(show_name no)
@@
 			)
 		)
-		(property "Footprint" ""
+		(property "Footprint" "TestPoint:TestPoint_Pad_D2.0mm"
 			(at 99.06 60.96 0)
 			(hide yes)
@@
 			(project "CycleSync"
 				(path "/3f2cc6af-e67b-48ad-b391-ff7619611bd8/5f3538da-ca0a-473f-9198-466d8964f21b"
-					(reference "TP2")
+					(reference "TP16")
 					(unit 1)
 				)
@@
 			)
 		)
-		(property "Footprint" ""
+		(property "Footprint" "Capacitor_SMD:C_1206_3216Metric"
 			(at 219.4052 35.56 0)
 			(hide yes)
@@
 			)
 		)
-		(property "Footprint" ""
+		(property "Footprint" "Capacitor_SMD:C_0402_1005Metric"
 			(at 207.9752 92.71 0)
 			(hide yes)
@@
 			)
 		)
-		(property "Footprint" ""
+		(property "Footprint" "Capacitor_SMD:C_0805_2012Metric"
 			(at 243.5352 92.71 0)
 			(hide yes)
@@
 			)
 		)
-		(property "Footprint" ""
+		(property "Footprint" "Resistor_SMD:R_0402_1005Metric"
 			(at 88.9 154.432 90)
 			(hide yes)
@@
 			)
 		)
-		(property "Footprint" ""
+		(property "Footprint" "Resistor_SMD:R_0402_1005Metric"
 			(at 113.792 100.33 90)
 			(hide yes)
@@
 			)
 		)
-		(property "Footprint" ""
+		(property "Footprint" "Resistor_SMD:R_0402_1005Metric"
 			(at 141.732 100.33 90)
 			(hide yes)
@@
 			)
 		)
-		(property "Footprint" ""
+		(property "Footprint" "Capacitor_SMD:C_0805_2012Metric"
 			(at 42.8752 166.37 0)
 			(hide yes)
@@
 		(dnp no)
 		(fields_autoplaced yes)
-		(property "Reference" "TP1"
+		(property "Reference" "TP15"
 			(at 80.01 58.293 0)
 			(show_name no)
@@
 			)
 		)
-		(property "Footprint" ""
+		(property "Footprint" "TestPoint:TestPoint_Pad_D2.0mm"
 			(at 82.55 62.23 0)
 			(hide yes)
@@
 			(project "CycleSync"
 				(path "/3f2cc6af-e67b-48ad-b391-ff7619611bd8/5f3538da-ca0a-473f-9198-466d8964f21b"
-					(reference "TP1")
+					(reference "TP15")
 					(unit 1)
 				)
@@
 			)
 		)
-		(property "Footprint" ""
+		(property "Footprint" "Resistor_SMD:R_0402_1005Metric"
 			(at 122.682 100.33 90)
 			(hide yes)
@@
 			)
 		)
-		(property "Footprint" ""
+		(property "Footprint" "Resistor_SMD:R_0402_1005Metric"
 			(at 121.92 154.432 90)
 			(hide yes)
@@
 			)
 		)
-		(property "Footprint" ""
+		(property "Footprint" "Capacitor_SMD:C_0402_1005Metric"
 			(at 195.2752 92.71 0)
 			(hide yes)
@@
 			)
 		)
-		(property "Footprint" ""
+		(property "Footprint" "Resistor_SMD:R_0402_1005Metric"
 			(at 142.24 57.658 90)
 			(hide yes)
@@
 		(dnp no)
 		(fields_autoplaced yes)
-		(property "Reference" "TP3"
+		(property "Reference" "TP17"
 			(at 110.49 57.023 0)
 			(show_name no)
@@
 			)
 		)
-		(property "Footprint" ""
+		(property "Footprint" "TestPoint:TestPoint_Pad_D2.0mm"
 			(at 113.03 60.96 0)
 			(hide yes)
@@
 			(project "CycleSync"
 				(path "/3f2cc6af-e67b-48ad-b391-ff7619611bd8/5f3538da-ca0a-473f-9198-466d8964f21b"
-					(reference "TP3")
+					(reference "TP17")
 					(unit 1)
 				)
@@
 		(dnp no)
 		(fields_autoplaced yes)
-		(property "Reference" "TP4"
+		(property "Reference" "TP18"
 			(at 125.73 57.023 0)
 			(show_name no)
@@
 			)
 		)
-		(property "Footprint" ""
+		(property "Footprint" "TestPoint:TestPoint_Pad_D2.0mm"
 			(at 128.27 60.96 0)
 			(hide yes)
@@
 			(project "CycleSync"
 				(path "/3f2cc6af-e67b-48ad-b391-ff7619611bd8/5f3538da-ca0a-473f-9198-466d8964f21b"
-					(reference "TP4")
+					(reference "TP18")
 					(unit 1)
 				)
@@
 			)
 		)
-		(property "Footprint" ""
+		(property "Footprint" "Capacitor_SMD:C_0805_2012Metric"
 			(at 247.3452 121.92 0)
 			(hide yes)

Commit message: added footprints and manufacturer part number
Parts:
- added TP24: GND_USB, TestPoint:TestPoint_Pad_D1.5mm, symbol Connector:TestPoint
- C51: Distributor Link (none) -> https://jlcpcb.com/partdetail/MurataElectronics-GRM155R71A1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; MANUFACTURER (none) -> Murata Electronics; MPN (none) -> GRM155R71A104KA01D
- C52, C53, C54, C67, C68: Distributor Link (none) -> https://jlcpcb.com/partdetail/236937-GRM21BZ71E106KE15L/C23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; MANUFACTURER (none) -> Murata Electronics; MPN (none) -> GRM21BZ71E106KE15L
- C55, C56: Distributor Link (none) -> https://jlcpcb.com/partdetail/13537-CL31A226KAHNNNE/C12891; MANUFACTURER (none) -> Samsung Electro-Mechanics; MPN (none) -> CL31A226KAHNNNE
- C57: Distributor Link (none) -> https://jlcpcb.com/partdetail/291005-CL05B104KB54PNC/C307331; MANUFACTURER (none) -> Samsung Electro-Mechanics; MPN (none) -> CL05B104KB54PNC
- C58, C59: Distributor Link (none) -> https://jlcpcb.com/partdetail/MurataElectronics-GRM1555C1H3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; MANUFACTURER (none) -> Murata Electronics; MPN (none) -> GRM1555C1H331JA01D
- C60, C61, C62, C63: Distributor Link (none) -> https://jlcpcb.com/partdetail/15869-CL05B103KB5NNNC/C15195; MANUFACTURER (none) -> Samsung Electro-Mechanics; MPN (none) -> CL05B103KB5NNNC
- C64: Distributor Link (none) -> https://jlcpcb.com/partdetail/2131-CL21A475KAQNNNE/C1779; MANUFACTURER (none) -> Samsung Electro-Mechanics; MPN (none) -> CL21A475KAQNNNE
- C65, C66: Distributor Link (none) -> https://jlcpcb.com/partdetail/TaiyoYuden-EMK325ABJ107MMT/C3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; MANUFACTURER (none) -> Taiyo Yuden; MPN (none) -> EMK325ABJ107MM-T
- R33, R34: Distributor Link (none) -> https://jlcpcb.com/partdetail/YAGEO-RC0402FR070RL/C106231; MANUFACTURER (none) -> YAGEO; MPN (none) -> RC0402FR-070RL
- R35, R38: Distributor Link (none) -> https://jlcpcb.com/partdetail/YAGEO-RC0402FR0710KL/C60490; MANUFACTURER (none) -> YAGEO; MPN (none) -> RC0402FR-0710KL
- R36, R37, R39, R40: Distributor Link (none) -> https://jlcpcb.com/partdetail/26622-0402WGF2201TCE/C25879; MANUFACTURER (none) -> UNI-ROYAL(Uniroyal Elec); MPN (none) -> 0402WGF2201TCE
- R41, R42: Distributor Link (none) -> https://jlcpcb.com/partdetail/26648-0402WGF5101TCE/C25905; MANUFACTURER (none) -> UNI-ROYAL(Uniroyal Elec); MPN (none) -> 0402WGF5101TCE
- R43, R44: Distributor Link (none) -> https://jlcpcb.com/partdetail/26648-0402WGF5101TCE/C25905; MANUFACTURER (none) -> UNI-ROYAL(Uniroyal Elec); MPN (none) -> 0402WGF5101TCE; now not fitted
- TP15, TP16, TP17, TP18: now left out of the parts list
- U7: Distributor Link (none) -> https://jlcpcb.com/partdetail/onsemi-CAT24C512WIGT3/C79986; MANUFACTURER (none) -> Onsemi; MPN (none) -> CAT24C512WI-GT3
- U8: Distributor Link (none) -> https://jlcpcb.com/partdetail/TexasInstruments-TPS25751DREF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; MANUFACTURER (none) -> Texas Instruments; MPN (none) -> TPS25751DREFR
- U9: value TVS2200DRV -> TVS2200DRVR; Distributor Link (none) -> https://jlcpcb.com/partdetail/TexasInstruments-TVS2200DRVR/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; MANUFACTURER (none) -> Texas Instruments; MPN (none) -> TVS2200DRV
Connections:
- net GND: now also TP24.1
